File: Hardware/analog-v10.brd (EAGLE design)
At the start: 100 x 80 mm, 50 parts, among them IC1 REG1117, Q1 LED ON, U1 ATMEGA328P, U10 QRE1113, U2 TB6612FNG, U3 QRE1113, U4 QRE1113, U5 QRE1113, U6 QRE1113, U7 QRE1113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

Commit message: Presentación de componentes
Parts:
- moved R17 190.0 mm to (129.5, 26.7), flipped to the bottom
- moved R4 161.1 mm to (100.3, 10.2)
- moved R2 154.6 mm to (100.3, 7.62)
- moved R6 149.7 mm to (129.5, 24.1), flipped to the bottom
- moved R3 147.7 mm to (95.2, 87.6), flipped to the bottom, turned to 180 degrees
- moved R15 141.2 mm to (90.2, 82.5), flipped to the bottom, turned to 180 degrees
- moved C1 140.1 mm to (81.3, 20.3), turned to 270 degrees
- moved C3 126.5 mm to (106.7, 44.5)
- moved R14 117.3 mm to (69.8, 82.5), flipped to the bottom, turned to 180 degrees
- moved R1 112.2 mm to (69.8, 68.6), flipped to the bottom
- moved R12 108.9 mm to (69.8, 76.2), flipped to the bottom
- moved R7 107.2 mm to (85.1, 87.6), flipped to the bottom
- moved R8 101.0 mm to (74.9, 87.6), flipped to the bottom, turned to 180 degrees
- moved R9 94.9 mm to (64.8, 87.6), flipped to the bottom, turned to 180 degrees
- moved R13 93.7 mm to (49.5, 82.5), flipped to the bottom, turned to 180 degrees
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Other:
- board size 100 x 80 mm -> 140 x 89.9 mm
