File: Hardware/contorno_clean.brd (EAGLE design)
At the start: 140 x 90 mm, 8 parts

Commit message: Presentación de componentes
Parts:
- removed E$1, E$2, E$3, E$4, E$5, E$6, E$7, E$8: (no value), SparkFun-Sensors:QRE1113
Other:
- board size 140 x 90 mm -> 140 x 89.9 mm
